Commit message: adjusted sdf to iiwa_description

File: src/demonstrator6_description/urdf/gripper.urdf.xacro (robot description, xacro)
@@ -2,5 +2,5 @@
 <robot xmlns:xacro="http://www.ros.org/wiki/xacro" name="prismatic_gripper">
   <joint name="base_link_joint" type="fixed">
-    <origin rpy="1.5707963705062866 -0 -0" xyz="0 0 0"/>
+    <origin rpy="1.5707963705062866 -0 -0" xyz="0 0 0.071"/>
     <parent link="iiwa_link_7"/>
     <child link="base_link_link"/>
@@ -31,5 +31,5 @@
     <inertial>
       <origin rpy="0 0 0" xyz="0 0 0"/>
-      <mass value="0.5"/>
+      <mass value="0.05"/>
       <inertia ixx="0.00017" ixy="0.0" ixz="0.0" iyy="0.0018" iyz="0.0" izz="0.0017"/>
     </inertial>
@@ -50,5 +50,5 @@
     <inertial>
       <origin rpy="0 0 0" xyz="0 0 0"/>
-      <mass value="0.1"/>
+      <mass value="0.01"/>
       <inertia ixx="0.0002" ixy="0.0" ixz="0.0" iyy="0.000195" iyz="0.0" izz="0.000021"/>
     </inertial>
@@ -69,5 +69,5 @@
     <inertial>
       <origin rpy="0 0 0" xyz="0 0 0"/>
-      <mass value="0.1"/>
+      <mass value="0.01"/>
       <inertia ixx="0.0002" ixy="0.0" ixz="0.0" iyy="0.000195" iyz="0.0" izz="0.000021"/>
     </inertial>
@@ -85,4 +85,13 @@
     </collision>
   </link>
+  <!--<gazebo reference="gripper_left_link">
+    <selfCollide>False</selfCollide>
+  </gazebo>
+  <gazebo reference="gripper_right_link">
+    <selfCollide>False</selfCollide>
+  </gazebo>
+  <gazebo reference="base_link_link">
+    <selfCollide>False</selfCollide>
+  </gazebo>-->
   <transmission name="gripper_tran_left">
     <robotNamespace>/iiwa</robotNamespace>

File: src/demonstrator6_description/urdf/iiwa_gripper.urdf (robot description, URDF)
Before this commit: robot iiwa_14, 9 links, 8 joints
Links:
- added link base_link_link, mass 0.05; collision mesh filename=package://demonstrator6_description/meshes/collision/COL_ba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 scale=1 1 1; visual mesh filename=package://demonstrator6_description/meshes/visual/VIS_base.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 scale=1 1 1
- added link gripper_left_link, mass 0.01; collision mesh filename=package://demonstrator6_description/meshes/collision/COL_gr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 scale=1 1 1; visual mesh filename=package://demonstrator6_description/meshes/visual/VIS_gripp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 scale=1 1 1
- added link gripper_right_link, mass 0.01; collision mesh filename=package://demonstrator6_description/meshes/collision/COL_gr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 scale=1 1 1; visual mesh filename=package://demonstrator6_description/meshes/visual/VIS_gripp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 scale=1 1 1
- added link iiwa_link_ee
- added link iiwa_link_ee_kuka
- added link iiwa_link_ee_kuka_mft_pneum
- link iiwa_link_0: geometry collision mesh filename=package://demonstrator6_description/meshes/iiwa14/collision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; visual mesh filename=package://demonstrator6_description/meshes/iiwa14/visual/li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
- link iiwa_link_1: geometry collision mesh filename=package://demonstrator6_description/meshes/iiwa14/collision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; visual mesh filename=package://demonstrator6_description/meshes/iiwa14/visual/li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
- link iiwa_link_2: geometry collision mesh filename=package://demonstrator6_description/meshes/iiwa14/collision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; visual mesh filename=package://demonstrator6_description/meshes/iiwa14/visual/li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
- link iiwa_link_3: geometry collision mesh filename=package://demonstrator6_description/meshes/iiwa14/collision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; visual mesh filename=package://demonstrator6_description/meshes/iiwa14/visual/li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
- link iiwa_link_4: geometry collision mesh filename=package://demonstrator6_description/meshes/iiwa14/collision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; visual mesh filename=package://demonstrator6_description/meshes/iiwa14/visual/li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
- link iiwa_link_5: geometry collision mesh filename=package://demonstrator6_description/meshes/iiwa14/collision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; visual mesh filename=package://demonstrator6_description/meshes/iiwa14/visual/li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
- link iiwa_link_6: geometry collision mesh filename=package://demonstrator6_description/meshes/iiwa14/collision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; visual mesh filename=package://demonstrator6_description/meshes/iiwa14/visual/li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
- link iiwa_link_7: geometry collision mesh filename=package://demonstrator6_description/meshes/iiwa14/collision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; visual mesh filename=package://demonstrator6_description/meshes/iiwa14/visual/li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
Joints:
- added joint base_link_joint: type fixed, parent iiwa_link_7, child base_link_link, origin xyz=0 0 0.071 rpy=1.5707963705062866 -0 -0, axis 0 0 1, limit lower=1.0 upper=1.0 effort=100.0 velocity=1.0
- added joint gripper_left_joint: type prismatic, parent base_link_link, child gripper_left_link, origin xyz=-0.0850000023841858 0.050000011920928955 0 rpy=1.5707963705062866 1.570796251296997 0, axis 0 1 0, limit lower=0.0 upper=0.0704 effort=100.0 velocity=1.0
- added joint gripper_right_joint: type prismatic, parent base_link_link, child gripper_right_link, origin xyz=0.0850000023841858 0.050000011920928955 0 rpy=1.5707963705062866 -1.570796251296997 0, axis 0 1 0, limit lower=0.0 upper=0.0704 effort=100.0 velocity=1.0
- added joint iiwa_joint_ee: type fixed, parent iiwa_link_7, child iiwa_link_ee, origin xyz=0 0 0.045 rpy=0 -1.57079632679 0
- added joint iiwa_joint_ee_kuka: type fixed, parent iiwa_link_7, child iiwa_link_ee_kuka, origin xyz=0 0 0.045 rpy=3.14159265359 3.14159265359 3.14159265359, axis 0 0 1
- added joint iiwa_joint_ee_kuka_mft_pneum: type fixed, parent iiwa_link_7, child iiwa_link_ee_kuka_mft_pneum, origin xyz=0 0 0.071 rpy=0 -1.57079632679 0
- joint iiwa_joint_7: origin xyz=0 0.181 0 rpy=-1.57079632679 3.14159265359 0 -> xyz=0 0.081 0 rpy=-1.57079632679 3.14159265359 0
- joint world_iiwa_joint: origin xyz=0 0 0 rpy=0 0 0 -> xyz=0 0 0.0 rpy=0 0 0

File: src/demonstrator6_description/urdf/iiwa_gripper.urdf.xacro (robot description, xacro)
@@ -1,5 +1,16 @@
 <?xml version="1.0"?>
 <robot xmlns:xacro="http://www.ros.org/wiki/xacro" name="iiwa14">
-  <xacro:include filename="$(find demonstrator6_description)/urdf/iiwa.urdf.xacro" />
+  <xacro:include filename="$(find demonstrator6_description)/urdf/materials.xacro" />
+  <!--Import the lbr iiwa macro -->
+  <xacro:include filename="$(find demonstrator6_description)/urdf/iiwa14.xacro"/>
+  <xacro:arg name="hardware_interface" default="EffortJointInterface"/>
+  <xacro:arg name="robot_name" default="iiwa"/>
+  <!-- Fix to world just for testing -->
+  <link name="world"/>
+  <!--iiwa-->
+  <xacro:iiwa14 hardware_interface="$(arg hardware_interface)" robot_name="$(arg robot_name)" parent="world">
+    <origin xyz="0 0 0.0" rpy="0 0 0" />
+  </xacro:iiwa14>
+<!--   <xacro:include filename="$(find demonstrator6_description)/urdf/iiwa.urdf.xacro" /> -->
   <xacro:include filename="$(find demonstrator6_description)/urdf/gripper.urdf.xacro" />
 </robot>

Commit message: update demonstrator6_description urdf

File: src/demonstrator6_description/urdf/gripper.urdf.xacro (robot description, xacro)
@@ -2,5 +2,5 @@
 <robot xmlns:xacro="http://www.ros.org/wiki/xacro" name="prismatic_gripper">
   <joint name="base_link_joint" type="fixed">
-    <origin rpy="1.5707963705062866 -0 -0" xyz="0 0 0.071"/>
+    <origin rpy="1.5707963705062866 -0 -0" xyz="0 0 0.045"/>
     <parent link="iiwa_link_7"/>
     <child link="base_link_link"/>
@@ -85,13 +85,4 @@
     </collision>
   </link>
-  <!--<gazebo reference="gripper_left_link">
-    <selfCollide>False</selfCollide>
-  </gazebo>
-  <gazebo reference="gripper_right_link">
-    <selfCollide>False</selfCollide>
-  </gazebo>
-  <gazebo reference="base_link_link">
-    <selfCollide>False</selfCollide>
-  </gazebo>-->
   <transmission name="gripper_tran_left">
     <robotNamespace>/iiwa</robotNamespace>

File: src/demonstrator6_description/urdf/iiwa14.xacro (robot description, xacro)
@@ -44,5 +44,5 @@
         <origin xyz="0 0 0" rpy="0 0 0"/>
         <geometry>
-          <mesh filename="package://demonstrator6_description/meshes/iiwa14/visual/link_0.stl"/>
+          <mesh filename="package://demonstrator6_description/meshes/visual/link_0.dae"/>
         </geometry>
         <material name="Grey"/>
@@ -51,5 +51,5 @@
         <origin xyz="0 0 0" rpy="0 0 0"/>
         <geometry>
-          <mesh filename="package://demonstrator6_description/meshes/iiwa14/collision/link_0_s.stl"/>
+          <mesh filename="package://demonstrator6_description/meshes/collision/link_0.dae"/>
         </geometry>
         <material name="Grey"/>
@@ -85,12 +85,12 @@
         <origin xyz="0 0 0" rpy="0 0 0"/>
         <geometry>
-          <mesh filename="package://demonstrator6_description/meshes/iiwa14/visual/link_1.stl"/>
-        </geometry>
-        <material name="Orange"/>
-      </visual>
-      <collision>
-        <origin xyz="0 0 0" rpy="0 0 0"/>
-        <geometry>
-          <mesh filename="package://demonstrator6_description/meshes/iiwa14/collision/link_1_s.stl"/>
+          <mesh filename="package://demonstrator6_description/meshes/visual/link_1.dae"/>
+        </geometry>
+        <material name="Orange"/>
+      </visual>
+      <collision>
+        <origin xyz="0 0 0" rpy="0 0 0"/>
+        <geometry>
+          <mesh filename="package://demonstrator6_description/meshes/collision/link_1.dae"/>
         </geometry>
         <material name="Orange"/>
@@ -120,12 +120,12 @@
         <origin xyz="0 0 0" rpy="0 0 0"/>
         <geometry>
-          <mesh filename="package://demonstrator6_description/meshes/iiwa14/visual/link_2.stl"/>
-        </geometry>
-        <material name="Orange"/>
-      </visual>
-      <collision>
-        <origin xyz="0 0 0" rpy="0 0 0"/>
-        <geometry>
-          <mesh filename="package://demonstrator6_description/meshes/iiwa14/collision/link_2_s.stl"/>
+          <mesh filename="package://demonstrator6_description/meshes/visual/link_2.dae"/>
+        </geometry>
+        <material name="Orange"/>
+      </visual>
+      <collision>
+        <origin xyz="0 0 0" rpy="0 0 0"/>
+        <geometry>
+          <mesh filename="package://demonstrator6_description/meshes/collision/link_2.dae"/>
         </geometry>
         <material name="Orange"/>
@@ -155,12 +155,12 @@
         <origin xyz="0 0 0" rpy="0 0 0"/>
         <geometry>
-          <mesh filename="package://demonstrator6_description/meshes/iiwa14/visual/link_3.stl"/>
-        </geometry>
-        <material name="Orange"/>
-      </visual>
-      <collision>
-        <origin xyz="0 0 0" rpy="0 0 0"/>
-        <geometry>
-          <mesh filename="package://demonstrator6_description/meshes/iiwa14/collision/link_3_s.stl"/>
+          <mesh filename="package://demonstrator6_description/meshes/visual/link_3.dae"/>
+        </geometry>
+        <material name="Orange"/>
+      </visual>
+      <collision>
+        <origin xyz="0 0 0" rpy="0 0 0"/>
+        <geometry>
+          <mesh filename="package://demonstrator6_description/meshes/collision/link_3.dae"/>
         </geometry>
         <material name="Orange"/>
@@ -190,12 +190,12 @@
         <origin xyz="0 0 0" rpy="0 0 0"/>
         <geometry>
-          <mesh filename="package://demonstrator6_description/meshes/iiwa14/visual/link_4.stl"/>
-        </geometry>
-        <material name="Orange"/>
-      </visual>
-      <collision>
-        <origin xyz="0 0 0" rpy="0 0 0"/>
-        <geometry>
-          <mesh filename="package://demonstrator6_description/meshes/iiwa14/collision/link_4_s.stl"/>
+          <mesh filename="package://demonstrator6_description/meshes/visual/link_4.dae"/>
+        </geometry>
+        <material name="Orange"/>
+      </visual>
+      <collision>
+        <origin xyz="0 0 0" rpy="0 0 0"/>
+        <geometry>
+          <mesh filename="package://demonstrator6_description/meshes/collision/link_4.dae"/>
         </geometry>
         <material name="Orange"/>
@@ -225,12 +225,12 @@
         <origin xyz="0 0 0" rpy="0 0 0"/>
         <geometry>
-          <mesh filename="package://demonstrator6_description/meshes/iiwa14/visual/link_5.stl"/>
-        </geometry>
-        <material name="Orange"/>
-      </visual>
-      <collision>
-        <origin xyz="0 0 0" rpy="0 0 0"/>
-        <geometry>
-          <mesh filename="package://demonstrator6_description/meshes/iiwa14/collision/link_5_s.stl"/>
+          <mesh filename="package://demonstrator6_description/meshes/visual/link_5.dae"/>
+        </geometry>
+        <material name="Orange"/>
+      </visual>
+      <collision>
+        <origin xyz="0 0 0" rpy="0 0 0"/>
+        <geometry>
+          <mesh filename="package://demonstrator6_description/meshes/collision/link_5.dae"/>
         </geometry>
         <material name="Orange"/>
@@ -260,12 +260,12 @@
         <origin xyz="0 0 0" rpy="0 0 0"/>
         <geometry>
-          <mesh filename="package://demonstrator6_description/meshes/iiwa14/visual/link_6.stl"/>
-        </geometry>
-        <material name="Orange"/>
-      </visual>
-      <collision>
-        <origin xyz="0 0 0" rpy="0 0 0"/>
-        <geometry>
-          <mesh filename="package://demonstrator6_description/meshes/iiwa14/collision/link_6_s.stl"/>
+          <mesh filename="package://demonstrator6_description/meshes/visual/link_6.dae"/>
+        </geometry>
+        <material name="Orange"/>
+      </visual>
+      <collision>
+        <origin xyz="0 0 0" rpy="0 0 0"/>
+        <geometry>
+          <mesh filename="package://demonstrator6_description/meshes/collision/link_6.dae"/>
         </geometry>
         <material name="Orange"/>
@@ -295,6 +295,5 @@
         <origin xyz="0 0 0" rpy="0 0 0"/>
         <geometry>
-<!--           <mesh filename="package://demonstrator6_description/meshes/iiwa14/visual/link_7.stl"/> -->
-		  <mesh filename="package://demonstrator6_description/meshes/iiwa14/visual/link_7-MF-Touch-pneumatisch.stl"/>
+          <mesh filename="package://demonstrator6_description/meshes/visual/link_7.dae"/>
         </geometry>
         <material name="Grey"/>
@@ -303,31 +302,8 @@
         <origin xyz="0 0 0" rpy="0 0 0"/>
         <geometry>
-<!--           <mesh filename="package://demonstrator6_description/meshes/iiwa14/collision/link_7_s.stl"/> -->
-		  <mesh filename="package://demonstrator6_description/meshes/iiwa14/collision/link_7-MF-Touch-pneumatisch_s.stl"/>
+          <mesh filename="package://demonstrator6_description/meshes/collision/link_7.dae"/>
         </geometry>
         <material name="Grey"/>
       </collision>
-    </link>
-    <joint name="${robot_name}_joint_ee" type="fixed">
-      <parent link="${robot_name}_link_7"/>
-      <child link="${robot_name}_link_ee"/>
-      <origin xyz="0 0 0.045" rpy="0 -${PI/2} 0"/>
-    </joint>
-    <link name="${robot_name}_link_ee">
-    </link>
-    <joint name="${robot_name}_joint_ee_kuka" type="fixed">
-      <parent link="${robot_name}_link_7"/>
-      <child link="${robot_name}_link_ee_kuka"/>
-      <origin xyz="0 0 0.045" rpy="${PI} ${PI} ${PI}"/>
-      <axis xyz="0 0 1"/>
-    </joint>
-	<joint name="${robot_name}_joint_ee_kuka_mft_pneum" type="fixed">
-      <parent link="${robot_name}_link_7"/>
-      <child link="${robot_name}_link_ee_kuka_mft_pneum"/>
-      <origin xyz="0 0 0.071" rpy="0 -${PI/2} 0"/>
-    </joint>
-    <link name="${robot_name}_link_ee_kuka">
-    </link>
-	<link name="${robot_name}_link_ee_kuka_mft_pneum">
     </link>
     <!--Extensions -->

File: src/demonstrator6_description/urdf/iiwa_gripper.urdf (robot description, URDF)
Before this commit: robot iiwa14, 15 links, 14 joints
Links:
- removed link iiwa_link_ee
- removed link iiwa_link_ee_kuka
- removed link iiwa_link_ee_kuka_mft_pneum
- link iiwa_link_0: geometry collision mesh filename=package://demonstrator6_description/meshes/collision/link_0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; visual mesh filename=package://demonstrator6_description/meshes/visual/link_0.dae
- link iiwa_link_1: geometry collision mesh filename=package://demonstrator6_description/meshes/collision/link_1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; visual mesh filename=package://demonstrator6_description/meshes/visual/link_1.dae
- link iiwa_link_2: geometry collision mesh filename=package://demonstrator6_description/meshes/collision/link_2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; visual mesh filename=package://demonstrator6_description/meshes/visual/link_2.dae
- link iiwa_link_3: geometry collision mesh filename=package://demonstrator6_description/meshes/collision/link_3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; visual mesh filename=package://demonstrator6_description/meshes/visual/link_3.dae
- link iiwa_link_4: geometry collision mesh filename=package://demonstrator6_description/meshes/collision/link_4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; visual mesh filename=package://demonstrator6_description/meshes/visual/link_4.dae
- link iiwa_link_5: geometry collision mesh filename=package://demonstrator6_description/meshes/collision/link_5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; visual mesh filename=package://demonstrator6_description/meshes/visual/link_5.dae
- link iiwa_link_6: geometry collision mesh filename=package://demonstrator6_description/meshes/collision/link_6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; visual mesh filename=package://demonstrator6_description/meshes/visual/link_6.dae
- link iiwa_link_7: geometry collision mesh filename=package://demonstrator6_description/meshes/collision/link_7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; visual mesh filename=package://demonstrator6_description/meshes/visual/link_7.dae
Joints:
- removed joint iiwa_joint_ee
- removed joint iiwa_joint_ee_kuka
- removed joint iiwa_joint_ee_kuka_mft_pneum
- joint base_link_joint: origin xyz=0 0 0.071 rpy=1.5707963705062866 -0 -0 -> xyz=0 0 0.045 rpy=1.5707963705062866 -0 -0
