Commit message: adjusted multiple robots urdf and changed ur5e gripper

File: src/demonstrator6_description/urdf/multiple_robots/multiple_robots.urdf.xacro (robot description, xacro)
@@ -2,29 +2,64 @@
 <robot name="multiple_robots"
        xmlns:xacro="http://www.ros.org/wiki/xacro">
-  <!--IIWA GRIPPER-->
+  <!--IIWA-->
   <xacro:include filename="$(find demonstrator6_description)/urdf/materials.xacro" />
-  <!--Import the lbr iiwa macro -->
   <xacro:include filename="$(find demonstrator6_description)/urdf/iiwa14.xacro"/>
   <xacro:arg name="hardware_interface" default="EffortJointInterface"/>
   <xacro:arg name="robot_name" default="iiwa"/>
-  <!--iiwa-->
   <xacro:iiwa14 hardware_interface="$(arg hardware_interface)" robot_name="$(arg robot_name)" parent="world">
-    <origin xyz="0 0 0.0" rpy="0 0 0" />
+    <origin xyz="0 0 0" rpy="0 0 0" />
   </xacro:iiwa14>
   <xacro:include filename="$(find demonstrator6_description)/urdf/gripper.urdf.xacro" />
-  <!--IIWA GRIPPER-->
+  <!--IIWA-->
   <!--PANDA-->
   <xacro:include filename="$(find franka_description)/robots/panda_arm.xacro"/>
   <xacro:include filename="$(find franka_description)/robots/hand.xacro"/>
-  <!-- for simulation -->
   <xacro:include filename="$(find franka_description)/robots/panda.gazebo.xacro"/>
   <xacro:include filename="$(find franka_description)/robots/panda.control.xacro"/>
-  <!-- end for simulation -->
   <xacro:panda_arm xyz="0 -5.0 0" rpy="0 0 0" connected_to="world" arm_id="panda"/>
   <xacro:hand ns="panda" rpy="0 0 ${-pi/4}" connected_to="panda_link8" safety_distance="0.03"/>
-  <!-- for simulation -->
   <xacro:panda_gazebo arm_id="panda"/>
   <xacro:panda_control arm_id="panda" load_hand="true" />
-  <!-- end for simulation -->
   <!--PANDA-->
+  <!--LWA4P-->
+  <xacro:include filename="$(find sacc_rec_grasp_description)/urdf/scene.gazebo.xacro" />
+  <link name ="arm_base_link"/>
+  <joint name="arm_base_joint" type="fixed">
+      <parent link="world" />
+      <child link = "arm_base_link" />
+      <origin xyz="0 -3.0 0" rpy="0 0 0" />
+  </joint>
+  <xacro:include filename="$(find schunk_description)/urdf/lwa4p/lwa4p.urdf.xacro" />
+  <xacro:schunk_lwa4p parent="arm_base_link" name="arm">
+      <origin xyz="0 0 0" rpy="0 0 0"/>
+      <xacro:property name="arm_1_ref" value="2.1" />
+      <xacro:property name="arm_2_ref" value="2.1" />
+      <xacro:property name="arm_3_ref" value="2.1" />
+      <xacro:property name="arm_4_ref" value="2.1" />
+      <xacro:property name="arm_5_ref" value="2.1" />
+      <xacro:property name="arm_6_ref" value="2.1" />
+  </xacro:schunk_lwa4p>
+  <xacro:include filename="$(find schunk_svh_description)/urdf/svh.urdf.xacro" />
+  <xacro:svh parent="arm_tcp_link" name="svh_hand" side="-1" robot_namespace="/svh/svh_ros_control_node">
+    <origin xyz="0 0 0"  rpy= "0 0 0" />
+  </xacro:svh>
+  <!--LWA4P-->
+  <!--UR5E-->
+  <xacro:include filename="$(find ur_e_description)/urdf/common.gazebo.xacro" />
+  <xacro:include filename="$(find ur_e_description)/urdf/ur5e.urdf.xacro" />
+  <xacro:ur5e_robot prefix="" joint_limited="true"
+    shoulder_pan_lower_limit="${-pi}" shoulder_pan_upper_limit="${pi}"
+    shoulder_lift_lower_limit="${-pi}" shoulder_lift_upper_limit="${pi}"
+    elbow_joint_lower_limit="${-pi}" elbow_joint_upper_limit="${pi}"
+    wrist_1_lower_limit="${-pi}" wrist_1_upper_limit="${pi}"
+    wrist_2_lower_limit="${-pi}" wrist_2_upper_limit="${pi}"
+    wrist_3_lower_limit="${-pi}" wrist_3_upper_limit="${pi}"
+  />
+  <joint name="world_joint" type="fixed">
+    <parent link="world" />
+    <child link = "base_link" />
+    <origin xyz="0.0 3.0 0.0" rpy="0.0 0.0 0.0" />
+  </joint>
+  <xacro:include filename="$(find demonstrator6_description)/urdf/ur5e/gripper_ur5e.urdf.xacro" />
+  <!--UR5E-->
 </robot>

File: src/demonstrator6_description/urdf/ur5e/ur5e_with_hand.urdf.xacro (robot description, xacro)
@@ -3,8 +3,4 @@
        xmlns:xacro="http://www.ros.org/wiki/xacro">
   <xacro:include filename="$(find ur_e_description)/urdf/ur5e_joint_limited_robot.urdf.xacro" />
-  <!-- load the SVH hand -->
-  <!--<xacro:include filename="$(find schunk_svh_description)/urdf/svh.urdf.xacro" />
-  <xacro:svh parent="tool0" name="svh_hand" side="-1" robot_namespace="/svh/svh_ros_control_node">
-    <origin xyz="0 0 0"  rpy= "0 0 0" />
-  </xacro:svh>-->
+  <xacro:include filename="$(find demonstrator6_description)/urdf/ur5e/gripper_ur5e.urdf.xacro" />
 </robot>
